Commit message: feat: activate SY205 URDF in backend

File: assets/model/kinematic_excavator.urdf (robot description, URDF)
Before this commit: robot kinematic_excavator, 13 links, 12 joints
Links:
- link arm_link: mass None -> 1290; geometry collision box size=0.419790009 1.189338999 3.943809109; visual box size=0.339790009 1.109338999 3.863809109
- link base_link: mass None -> 9460; geometry collision box size=3.067423897 4.325371103 0.978877971; visual box size=2.987423897 4.245371103 0.898877971
- link boom_link: mass None -> 2150; geometry collision box size=0.682465004 4.184796976 4.70371695; visual box size=0.602465004 4.104796976 4.62371695
- link bucket_link: mass None -> 860; geometry collision box size=1.391366022 1.30420907 1.673720913; visual box size=1.311366022 1.22420907 1.593720913
- link tooth_center: geometry visual sphere radius=0.03
- link tooth_left: geometry visual sphere radius=0.03
- link tooth_right: geometry visual sphere radius=0.03
- link upper_structure_link: mass None -> 7740; geometry collision box size=3.238524036 4.445462899 2.609148996; visual box size=3.158524036 4.365462899 2.529148996
Joints:
- joint arm_imu_joint: origin xyz=0 1.244230565 0 rpy=0 0 0 -> xyz=-0.000820003 0.163279414 -1.249701738 rpy=0 0 0
- joint arm_joint: origin xyz=0 4.67108234 0 rpy=4.869468613064179 0 0 -> xyz=0.066 -3.915 4.295 rpy=0 0 0
- joint boom_imu_joint: origin xyz=0 2.33554117 0 rpy=0 0 0 -> xyz=0.004933506 -1.972438484 2.159274399 rpy=0 0 0
- joint boom_joint: origin xyz=0.11134509 0.10503961 -1.15396138 rpy=0.6283185307179586 0 0 -> xyz=-0.119 0.075 0.713 rpy=0 0 0
- joint bucket_imu_joint: origin xyz=0 0.605347915 0 rpy=0 0 0 -> xyz=0.005774003 0.5036515 0.36291647 rpy=0 0 0
- joint bucket_joint: origin xyz=0 2.48846113 0 rpy=5.672320068981572 0 0 -> xyz=-0.008 0.63 -3.026 rpy=0 0 0
- joint gnss_joint: origin xyz=1.05304 -1.6763 -0.0 rpy=0 0 0 -> xyz=0 0.740756452 2.07440697 rpy=0 0 0
- joint swing_imu_joint: origin xyz=0 0 0.45 rpy=0 0 0 -> xyz=0 0.740756452 0.759832472 rpy=0 0 0
- joint swing_joint: origin xyz=0 0 1.55 rpy=0 0 0 -> xyz=0 0 0.91 rpy=0 0 0
- joint tooth_center_joint: origin xyz=0 1.21069583 0 rpy=0 0 0 -> xyz=0.00095452 1.114953041 0.216117024 rpy=0 0 0
- joint tooth_left_joint: origin xyz=-0.4775 1.21069583 0 rpy=0 0 0 -> xyz=-0.590063978 1.114150047 0.219933033 rpy=0 0 0
- joint tooth_right_joint: origin xyz=0.4775 1.21069583 0 rpy=0 0 0 -> xyz=0.591973018 1.115756035 0.212301016 rpy=0 0 0
