Commit message: feat(sy155w): drop arm four-bar, extend stick +30deg, pin pad-tilt regression
- import_sy155w: remove BUCKET_ROCKER/BUCKET_COUPLER subtrees with the bucket
  tree; BUCKET_CYLINDER rod now pins BUCKET_JOINT directly (horn pin
  0.22/0/0.26); arm_joint limit widened to [-9,+39] deg (+30 deg extension);
  source-pose oracle drops the direct-drive cylinder (no source oracle exists
  for the new pin geometry) along with the removed linkage nodes
- passive_hydraulics: no four_bar block in the manifest; cylinders still
  pin-follow and reject non-planar pins atomically
- sy155w_import_test: asserts linkage absence, sweeps arm to +39, and keeps
  atomic-retention via a non-planar pin displacement
- sy155w_session_test: new end-to-end gamepad regression - D-pad Down +
  right-stick Y/X must drive XTR13 tilt/rotate through the real
  InputMap -> MotionClient -> ProductSession -> AttachmentRig path while the
  boom/bucket base axes stay masked (the reported "tilt only curls the bucket"
  symptom reproduces only on builds predating pad-layer commit 4c95a32)
- spec: record the removed-linkage contract, direct-drive pins, widened arm
  limit, and the stale .godot/imported GLB cache lesson
- regenerated: runtime GLB, visual manifest, physics rig, parity fixture,
  source-pose oracle, URDF, evidence, provenance, catalog sha pins

Generated with [Devin](https://devin.ai)

Co-Authored-By: Devin <158243242+devin-ai-integration[bot]@users.noreply.github.com>

File: assets/model/library/sy155w_reference.urdf (robot description, URDF)
Before this commit: robot sy155w, 13 links, 12 joints
Joints:
- joint arm_joint: limit lower=-0.15707963267948966 upper=0.15707963267948966 effort=1000000 velocity=1 -> lower=-0.15707963267948966 upper=0.6806784082777885 effort=1000000 velocity=1

Commit message: feat(sy155w): widen bucket joint limits to +-40 deg
Both sides of bucket_joint gain 25 deg over the demonstrated source
range ([-15,+15] -> [-40,+40]) at user request; the carry-pose seed
(-10 deg) stays inside the new band. Import test sweeps the new
extremes.

Generated with [Devin](https://devin.ai)

Co-Authored-By: Devin <158243242+devin-ai-integration[bot]@users.noreply.github.com>

File: assets/model/library/sy155w_reference.urdf (robot description, URDF)
Before this commit: robot sy155w, 13 links, 12 joints
Joints:
- joint bucket_joint: limit lower=-0.2617993877991494 upper=0.2617993877991494 effort=1000000 velocity=1 -> lower=-0.6981317007977318 upper=0.6981317007977318 effort=1000000 velocity=1

Commit message: feat(sy155w): widen boom limits, strip bucket-cylinder mounts
boom_joint gains +15 deg lower / +10 deg raise ([-7,+7] -> [-22,+17]);
the carry seed (+6) stays inside. The deleted cylinder's welded base
ears and pin on the stick are removed too (75 nodes stripped in total).
Import test sweeps the new extremes and asserts the mounts are absent.

Generated with [Devin](https://devin.ai)

Co-Authored-By: Devin <158243242+devin-ai-integration[bot]@users.noreply.github.com>

File: assets/model/library/sy155w_reference.urdf (robot description, URDF)
Before this commit: robot sy155w, 13 links, 12 joints
Joints:
- joint boom_joint: limit lower=-0.12217304763960307 upper=0.12217304763960307 effort=1000000 velocity=1 -> lower=-0.3839724354387525 upper=0.29670597283903605 effort=1000000 velocity=1
